File: SAO board.kicad_pcb (KiCad board)
At the start: 2 copper layers, 210 x 297 mm, 44 parts, among them J1 5V, SW1 SW_SPDT, U1 MIC5219-3.3YM5, U2 MIC5219-3.3YM5, U3 MIC5219-3.3YM5, U4 MIC5219-3.3YM5, U5 MIC5219-3.3YM5

Commit message: updated circuit and layout
Parts:
- added J10: Conn_01x01_Pin, Connector_PinHeader_2.54mm:PinHeader_1x01_P2.54mm_Horizontal, F.Cu at (51.6, 66.0)
- added J11: Conn_01x01_Pin, Connector_PinHeader_2.54mm:PinHeader_1x01_P2.54mm_Horizontal, F.Cu at (240.6, 123.0)
- added J12: Conn_01x01_Pin, Connector_PinHeader_2.54mm:PinHeader_1x01_P2.54mm_Horizontal, F.Cu at (241.0, 137.0)
- added J13: Conn_01x01_Pin, Connector_PinHeader_2.54mm:PinHeader_1x01_P2.54mm_Horizontal, F.Cu at (177.6, 135.0)
- added J14: Conn_01x01_Pin, Connector_PinHeader_2.54mm:PinHeader_1x01_P2.54mm_Horizontal, F.Cu at (178.6, 123.0)
- added J15: Conn_01x01_Pin, Connector_PinHeader_2.54mm:PinHeader_1x01_P2.54mm_Horizontal, F.Cu at (114.6, 121.0)
- added J16: Conn_01x01_Pin, Connector_PinHeader_2.54mm:PinHeader_1x01_P2.54mm_Horizontal, F.Cu at (115.6, 137.0)
- added J17: Conn_01x01_Pin, Connector_PinHeader_2.54mm:PinHeader_1x01_P2.54mm_Horizontal, F.Cu at (51.0, 135.0)
- added J18: Conn_01x01_Pin, Connector_PinHeader_2.54mm:PinHeader_1x01_P2.54mm_Horizontal, F.Cu at (51.6, 124.0)
- added J19: Conn_01x01_Pin, Connector_PinHeader_2.54mm:PinHeader_1x01_P2.54mm_Horizontal, F.Cu at (51.6, 194.0)
- added J2: ~, Connector_PinHeader_2.54mm:PinHeader_1x02_P2.54mm_Vertical, F.Cu at (111.0, 319.0)
- added J20: Conn_01x01_Pin, Connector_PinHeader_2.54mm:PinHeader_1x01_P2.54mm_Horizontal, F.Cu at (51.6, 206.0)
- added J21: Conn_01x01_Pin, Connector_PinHeader_2.54mm:PinHeader_1x01_P2.54mm_Horizontal, F.Cu at (111.6, 206.0)
- added J22: Conn_01x01_Pin, Connector_PinHeader_2.54mm:PinHeader_1x01_P2.54mm_Horizontal, F.Cu at (110.6, 194.0)
- added J23: Conn_01x01_Pin, Connector_PinHeader_2.54mm:PinHeader_1x01_P2.54mm_Horizontal, F.Cu at (177.6, 194.0)
- added J24: Conn_01x01_Pin, Connector_PinHeader_2.54mm:PinHeader_1x01_P2.54mm_Horizontal, F.Cu at (178.6, 205.0)
- added J25: Conn_01x01_Pin, Connector_PinHeader_2.54mm:PinHeader_1x01_P2.54mm_Horizontal, F.Cu at (241.6, 206.0)
- added J26: Conn_01x01_Pin, Connector_PinHeader_2.54mm:PinHeader_1x01_P2.54mm_Horizontal, F.Cu at (240.6, 193.0)
- added J27: Conn_01x01_Pin, Connector_PinHeader_2.54mm:PinHeader_1x01_P2.54mm_Horizontal, F.Cu at (240.6, 243.0)
- added J28: Conn_01x01_Pin, Connector_PinHeader_2.54mm:PinHeader_1x01_P2.54mm_Horizontal, F.Cu at (241.6, 256.0)
- added J29: Conn_01x01_Pin, Connector_PinHeader_2.54mm:PinHeader_1x01_P2.54mm_Horizontal, F.Cu at (178.6, 255.0)
- added J3: Conn_01x01_Pin, Connector_PinHeader_2.54mm:PinHeader_1x01_P2.54mm_Horizontal, F.Cu at (240.6, 65.0)
- added J30: Conn_01x01_Pin, Connector_PinHeader_2.54mm:PinHeader_1x01_P2.54mm_Horizontal, F.Cu at (177.6, 244.0)
- added J31: Conn_01x01_Pin, Connector_PinHeader_2.54mm:PinHeader_1x01_P2.54mm_Horizontal, F.Cu at (111.6, 255.0)
- added J32: Conn_01x01_Pin, Connector_PinHeader_2.54mm:PinHeader_1x01_P2.54mm_Horizontal, F.Cu at (111.6, 243.0)
- added J33: Conn_01x01_Pin, Connector_PinHeader_2.54mm:PinHeader_1x01_P2.54mm_Horizontal, F.Cu at (50.6, 243.0)
- added J34: Conn_01x01_Pin, Connector_PinHeader_2.54mm:PinHeader_1x01_P2.54mm_Horizontal, F.Cu at (50.6, 255.0)
- added J35: Conn_01x01_Pin, Connector_PinHeader_2.54mm:PinHeader_1x01_P2.54mm_Horizontal, F.Cu at (240.6, 294.0)
- added J36: Conn_01x01_Pin, Connector_PinHeader_2.54mm:PinHeader_1x01_P2.54mm_Horizontal, F.Cu at (240.6, 305.0)
- added J37: Conn_01x01_Pin, Connector_PinHeader_2.54mm:PinHeader_1x01_P2.54mm_Horizontal, F.Cu at (178.6, 305.0)
- added J38: Conn_01x01_Pin, Connector_PinHeader_2.54mm:PinHeader_1x01_P2.54mm_Horizontal, F.Cu at (177.6, 294.0)
- added J39: Conn_01x01_Pin, Connector_PinHeader_2.54mm:PinHeader_1x01_P2.54mm_Horizontal, F.Cu at (111.6, 293.0)
- added J4: Conn_01x01_Pin, Connector_PinHeader_2.54mm:PinHeader_1x01_P2.54mm_Horizontal, F.Cu at (239.6, 55.0)
- added J40: Conn_01x01_Pin, Connector_PinHeader_2.54mm:PinHeader_1x01_P2.54mm_Horizontal, F.Cu at (110.6, 305.0)
- added J41: Conn_01x01_Pin, Connector_PinHeader_2.54mm:PinHeader_1x01_P2.54mm_Horizontal, F.Cu at (51.6, 293.0)
- added J42: Conn_01x01_Pin, Connector_PinHeader_2.54mm:PinHeader_1x01_P2.54mm_Horizontal, F.Cu at (51.6, 304.0)
- added J5: Conn_01x01_Pin, Connector_PinHeader_2.54mm:PinHeader_1x01_P2.54mm_Horizontal, F.Cu at (173.6, 53.0)
- added J6: Conn_01x01_Pin, Connector_PinHeader_2.54mm:PinHeader_1x01_P2.54mm_Horizontal, F.Cu at (174.0, 68.0)
- added J7: Conn_01x01_Pin, Connector_PinHeader_2.54mm:PinHeader_1x01_P2.54mm_Horizontal, F.Cu at (114.0, 66.0)
- added J8: Conn_01x01_Pin, Connector_PinHeader_2.54mm:PinHeader_1x01_P2.54mm_Horizontal, F.Cu at (114.6, 52.0)
- added J9: Conn_01x01_Pin, Connector_PinHeader_2.54mm:PinHeader_1x01_P2.54mm_Horizontal, F.Cu at (50.6, 53.0)
- added R3: 4.7K, Inductor_SMD:L_1008_2520Metric, F.Cu at (63.1, 91.0)
- SAO-00, SAO-01, SAO-02, SAO-04, SAO-05, SAO-06, SAO-07, SAO-08, SAO-09, SAO-10, SAO-11, SAO-12, SAO-13, SAO-14, SAO-15, SAO-16, SAO-17, SAO-18, SAO-19: value Conn_02x03_Odd_Even -> SAO
- SAO-03: value ~ -> SAO
- moved D1 8.05 mm to (99.1, 314.0)
- moved R1 8.05 mm to (99.1, 323.0)
- moved SW1 6.18 mm to (60.0, 322.0)
- moved J1 6.08 mm to (80.5, 322.5)
Connections:
- net Net-(D1-K) renamed GND
- C7 pad 1: Net-(SAO-04-Pin_1) -> Net-(SAO-05-Vcc)
- R2 pad 2: Net-(SAO-00-Pin_3) -> Net-(J2-Pin_2)
- SAO-00 pad 3: Net-(SAO-00-Pin_3) -> Net-(J2-Pin_1)
- SAO-00 pad 4: Net-(SAO-00-Pin_4) -> Net-(J2-Pin_2)
- SAO-00 pad 5: unconnected-(SAO-00-Pin_5-Pad5) -> Net-(J10-Pin_1)
- SAO-00 pad 6: unconnected-(SAO-00-Pin_6-Pad6) -> Net-(J9-Pin_1)
- SAO-01 pad 3: Net-(SAO-00-Pin_3) -> Net-(J2-Pin_1)
- SAO-01 pad 4: Net-(SAO-00-Pin_4) -> Net-(J2-Pin_2)
- SAO-01 pad 5: unconnected-(SAO-01-Pin_5-Pad5) -> Net-(J7-Pin_1)
- SAO-01 pad 6: unconnected-(SAO-01-Pin_6-Pad6) -> Net-(J8-Pin_1)
- SAO-02 pad 3: Net-(SAO-00-Pin_3) -> Net-(J2-Pin_1)
- SAO-02 pad 4: Net-(SAO-00-Pin_4) -> Net-(J2-Pin_2)
- SAO-02 pad 5: unconnected-(SAO-02-Pin_5-Pad5) -> Net-(J6-Pin_1)
- SAO-02 pad 6: unconnected-(SAO-02-Pin_6-Pad6) -> Net-(J5-Pin_1)
- SAO-03 pad 3: Net-(SAO-00-Pin_3) -> Net-(J2-Pin_1)
- SAO-03 pad 4: Net-(SAO-00-Pin_4) -> Net-(J2-Pin_2)
- SAO-03 pad 5: unconnected-(SAO-03-Pin_5-Pad5) -> Net-(J3-Pin_1)
- SAO-03 pad 6: unconnected-(SAO-03-Pin_6-Pad6) -> Net-(J4-Pin_1)
- SAO-04 pad 1: Net-(SAO-04-Pin_1) -> unconnected-(SAO-04-Vcc-Pad1)
- SAO-04 pad 3: Net-(SAO-00-Pin_3) -> Net-(J2-Pin_1)
- SAO-04 pad 4: Net-(SAO-00-Pin_4) -> Net-(J2-Pin_2)
- SAO-04 pad 5: unconnected-(SAO-04-Pin_5-Pad5) -> Net-(J17-Pin_1)
- SAO-04 pad 6: unconnected-(SAO-04-Pin_6-Pad6) -> Net-(J18-Pin_1)
- SAO-05 pad 1: Net-(SAO-04-Pin_1) -> Net-(SAO-05-Vcc)
- SAO-05 pad 3: Net-(SAO-00-Pin_3) -> Net-(J2-Pin_1)
- SAO-05 pad 4: Net-(SAO-00-Pin_4) -> Net-(J2-Pin_2)
- SAO-05 pad 5: unconnected-(SAO-05-Pin_5-Pad5) -> Net-(J16-Pin_1)
- SAO-05 pad 6: unconnected-(SAO-05-Pin_6-Pad6) -> Net-(J15-Pin_1)
- SAO-06 pad 1: Net-(SAO-04-Pin_1) -> Net-(SAO-05-Vcc)
- SAO-06 pad 3: Net-(SAO-00-Pin_3) -> Net-(J2-Pin_1)
- SAO-06 pad 4: Net-(SAO-00-Pin_4) -> Net-(J2-Pin_2)
- SAO-06 pad 5: unconnected-(SAO-06-Pin_5-Pad5) -> Net-(J13-Pin_1)
- SAO-06 pad 6: unconnected-(SAO-06-Pin_6-Pad6) -> Net-(J14-Pin_1)
- SAO-07 pad 1: Net-(SAO-04-Pin_1) -> Net-(SAO-05-Vcc)
- SAO-07 pad 3: Net-(SAO-00-Pin_3) -> Net-(J2-Pin_1)
- SAO-07 pad 4: Net-(SAO-00-Pin_4) -> Net-(J2-Pin_2)
- SAO-07 pad 5: unconnected-(SAO-07-Pin_5-Pad5) -> Net-(J12-Pin_1)
- SAO-07 pad 6: unconnected-(SAO-07-Pin_6-Pad6) -> Net-(J11-Pin_1)
- SAO-08 pad 3: Net-(SAO-00-Pin_3) -> Net-(J2-Pin_1)
- SAO-08 pad 4: Net-(SAO-00-Pin_4) -> Net-(J2-Pin_2)
- SAO-08 pad 5: unconnected-(SAO-08-Pin_5-Pad5) -> Net-(J20-Pin_1)
- SAO-08 pad 6: unconnected-(SAO-08-Pin_6-Pad6) -> Net-(J19-Pin_1)
- SAO-09 pad 3: Net-(SAO-00-Pin_3) -> Net-(J2-Pin_1)
- SAO-09 pad 4: Net-(SAO-00-Pin_4) -> Net-(J2-Pin_2)
- SAO-09 pad 5: unconnected-(SAO-09-Pin_5-Pad5) -> Net-(J21-Pin_1)
- SAO-09 pad 6: unconnected-(SAO-09-Pin_6-Pad6) -> Net-(J22-Pin_1)
- SAO-10 pad 3: Net-(SAO-00-Pin_3) -> Net-(J2-Pin_1)
- SAO-10 pad 4: Net-(SAO-00-Pin_4) -> Net-(J2-Pin_2)
- SAO-10 pad 5: unconnected-(SAO-10-Pin_5-Pad5) -> Net-(J24-Pin_1)
- SAO-10 pad 6: unconnected-(SAO-10-Pin_6-Pad6) -> Net-(J23-Pin_1)
- SAO-11 pad 3: Net-(SAO-00-Pin_3) -> Net-(J2-Pin_1)
- SAO-11 pad 4: Net-(SAO-00-Pin_4) -> Net-(J2-Pin_2)
- SAO-11 pad 5: unconnected-(SAO-11-Pin_5-Pad5) -> Net-(J25-Pin_1)
- SAO-11 pad 6: unconnected-(SAO-11-Pin_6-Pad6) -> Net-(J26-Pin_1)
- SAO-12 pad 3: Net-(SAO-00-Pin_3) -> Net-(J2-Pin_1)
- SAO-12 pad 4: Net-(SAO-00-Pin_4) -> Net-(J2-Pin_2)
- SAO-12 pad 5: unconnected-(SAO-12-Pin_5-Pad5) -> Net-(J34-Pin_1)
- SAO-12 pad 6: unconnected-(SAO-12-Pin_6-Pad6) -> Net-(J33-Pin_1)
- SAO-13 pad 3: Net-(SAO-00-Pin_3) -> Net-(J2-Pin_1)
- SAO-13 pad 4: Net-(SAO-00-Pin_4) -> Net-(J2-Pin_2)
- SAO-13 pad 5: unconnected-(SAO-13-Pin_5-Pad5) -> Net-(J31-Pin_1)
- SAO-13 pad 6: unconnected-(SAO-13-Pin_6-Pad6) -> Net-(J32-Pin_1)
- SAO-14 pad 3: Net-(SAO-00-Pin_3) -> Net-(J2-Pin_1)
- SAO-14 pad 4: Net-(SAO-00-Pin_4) -> Net-(J2-Pin_2)
- SAO-14 pad 5: unconnected-(SAO-14-Pin_5-Pad5) -> Net-(J29-Pin_1)
- SAO-14 pad 6: unconnected-(SAO-14-Pin_6-Pad6) -> Net-(J30-Pin_1)
- SAO-15 pad 3: Net-(SAO-00-Pin_3) -> Net-(J2-Pin_1)
- SAO-15 pad 4: Net-(SAO-00-Pin_4) -> Net-(J2-Pin_2)
- SAO-15 pad 5: unconnected-(SAO-15-Pin_5-Pad5) -> Net-(J28-Pin_1)
- SAO-15 pad 6: unconnected-(SAO-15-Pin_6-Pad6) -> Net-(J27-Pin_1)
- SAO-16 pad 3: Net-(SAO-00-Pin_3) -> Net-(J2-Pin_1)
- SAO-16 pad 4: Net-(SAO-00-Pin_4) -> Net-(J2-Pin_2)
- SAO-16 pad 5: unconnected-(SAO-16-Pin_5-Pad5) -> Net-(J42-Pin_1)
- SAO-16 pad 6: unconnected-(SAO-16-Pin_6-Pad6) -> Net-(J41-Pin_1)
- SAO-17 pad 3: Net-(SAO-00-Pin_3) -> Net-(J2-Pin_1)
- SAO-17 pad 4: Net-(SAO-00-Pin_4) -> Net-(J2-Pin_2)
- SAO-17 pad 5: unconnected-(SAO-17-Pin_5-Pad5) -> Net-(J40-Pin_1)
- SAO-17 pad 6: unconnected-(SAO-17-Pin_6-Pad6) -> Net-(J39-Pin_1)
- SAO-18 pad 3: Net-(SAO-00-Pin_3) -> Net-(J2-Pin_1)
- SAO-18 pad 4: Net-(SAO-00-Pin_4) -> Net-(J2-Pin_2)
- SAO-18 pad 5: unconnected-(SAO-18-Pin_5-Pad5) -> Net-(J37-Pin_1)
- SAO-18 pad 6: unconnected-(SAO-18-Pin_6-Pad6) -> Net-(J38-Pin_1)
- SAO-19 pad 3: Net-(SAO-00-Pin_3) -> Net-(J2-Pin_1)
- SAO-19 pad 4: Net-(SAO-00-Pin_4) -> Net-(J2-Pin_2)
- SAO-19 pad 5: unconnected-(SAO-19-Pin_5-Pad5) -> Net-(J36-Pin_1)
- SAO-19 pad 6: unconnected-(SAO-19-Pin_6-Pad6) -> Net-(J35-Pin_1)
- U2 pad 5: Net-(SAO-04-Pin_1) -> Net-(SAO-05-Vcc)
